Commit message: Adapted positions to new viewer, Add script for HRP2 just moving his hand

File: urdf/walls.urdf (robot description, URDF)
Before this commit: robot walls, 5 links, 4 joints
Links:
- link l_wall_four: geometry collision box size=.01 6 2.5; visual box size=.01 6 2.5
- link l_wall_one: geometry collision box size=.01 6 2.5; visual box size=.01 6 2.5
- link l_wall_three: geometry collision box size=.01 6 1.2; visual box size=.01 6 1.2
- link l_wall_two: geometry collision box size=.01 6 2.5; visual box size=.01 6 2.5
- link wall_base: geometry visual box size=6 6 0.01
