Commit message: Add wood shelf

File: urdf/room.urdf (robot description, URDF)
Before this commit: robot room, 12 links, 11 joints
Links:
- link stuff_base: geometry collision mesh filename=package://room_description/meshes/etagere_bois_sized2.dae; visual mesh filename=package://room_description/meshes/etagere_bois_sized2.dae

Commit message: Update of urdf file

File: urdf/room.urdf (robot description, URDF)
Before this commit: robot room, 12 links, 11 joints
Links:
- link armchair_base: mass 1.0 -> None
- link beer_base: mass 1.0 -> None
- link books_base: mass 1.0 -> None
- link chair_base: mass 1.0 -> None
- link commode_base: mass 1.0 -> None
- link deskLamp_base: mass 1.0 -> None
- link desk_base: mass 1.0 -> None
- link lamp_base: mass 1.0 -> None
- link pc_base: mass 1.0 -> None
- link room_base: mass 1.0 -> None
- link stuff_base: mass 1.0 -> None
- link table_base: mass 1.0 -> None; geometry collision box size=0.9 1.5 0.3; visual box size=0.9 1.5 0.3

Commit message: Better meshes or textures in the room, meshes for walls and floor

File: urdf/room.urdf (robot description, URDF)
Before this commit: robot room, 12 links, 11 joints
Links:
- added link l_carpet; collision mesh filename=package://room_description/meshes/carpet.dae; visual mesh filename=package://room_description/meshes/carpet.dae
- added link l_carpet_wall_one, mass 1.0; collision mesh filename=package://room_description/meshes/wall_carpet.dae; visual mesh filename=package://room_description/meshes/wall_carpet.dae
- added link l_carpet_wall_two, mass 1.0; collision mesh filename=package://room_description/meshes/wall_carpet.dae; visual mesh filename=package://room_description/meshes/wall_carpet.dae
- link desk_base: geometry collision mesh filename=package://room_description/meshes/bureau_angulaire.dae; visual mesh filename=package://room_description/meshes/bureau_angulaire.dae
- link stuff_base: geometry collision mesh filename=package://room_description/meshes/etagere_bois2.dae; visual mesh filename=package://room_description/meshes/etagere_bois2.dae
- link table_base: geometry collision mesh filename=package://room_description/meshes/table_basse_truquee.dae; visual mesh filename=package://room_description/meshes/table_basse_truquee.dae
Joints:
- added joint j_carpet: type fixed, parent room_base, child l_carpet, origin xyz=0 0 0 rpy=0 0 0
- added joint j_carpet_wall_one: type fixed, parent room_base, child l_carpet_wall_one, origin xyz=0 0 0 rpy=0 0 0
- added joint j_carpet_wall_two: type fixed, parent room_base, child l_carpet_wall_two, origin xyz=0 0 0 rpy=0 0 0

File: urdf/walls.urdf (robot description, URDF)
Before this commit: robot walls, 5 links, 4 joints
Links:
- removed link l_wall_three
- removed link l_wall_two
- added link l_wall_roof, mass 1.0; collision box size=6 6 0.05; visual box size=6 6 0.05
- link wall_base: geometry visual box size=0.01 0.01 0.01
Joints:
- removed joint j_wall_three
- removed joint j_wall_two
- added joint j_wall_roof: type fixed, parent wall_base, child l_wall_roof, origin xyz=0 0 0 rpy=0 0 0

Commit message: Remove collision part of box base in room.urdf

File: urdf/room.urdf (robot description, URDF)
Before this commit: robot room, 15 links, 14 joints
Links:
- link room_base: geometry visual box size=0.01 0.01 0.01

Commit message: Add meshes, skeleton robot

File: urdf/room.urdf (robot description, URDF)
Before this commit: robot room, 15 links, 14 joints
Links:
- added link l_box_shelf_1, mass 1.0; collision box size=0.6 0.18 0.04; visual box size=0.6 0.18 0.04
- added link l_box_shelf_2, mass 1.0; collision box size=0.56 0.18 0.04; visual box size=0.56 0.18 0.04
- added link l_box_shelf_3, mass 1.0; collision box size=0.6 0.18 0.04; visual box size=0.6 0.18 0.04
- added link l_box_shelf_4, mass 1.0; collision box size=0.6 0.18 0.04; visual box size=0.6 0.18 0.04
Joints:
- added joint j_box_shelf_1: type fixed, parent room_base, child l_box_shelf_1, origin xyz=0 0 0 rpy=0 0 0
- added joint j_box_shelf_2: type fixed, parent room_base, child l_box_shelf_2, origin xyz=0 0 0 rpy=0 0 0
- added joint j_box_shelf_3: type fixed, parent room_base, child l_box_shelf_3, origin xyz=0 0 0 rpy=0 0 0
- added joint j_box_shelf_4: type fixed, parent room_base, child l_box_shelf_4, origin xyz=0 0 0 rpy=0 0 0
